Commit message: Getting the RTAB-Map node to work

File: src/my_robot/urdf/my_robot.xacro (robot description, xacro)
@@ -154,4 +154,12 @@
     <dynamics damping="1.0" friction="1.0"/>
   </joint>
+  <!-- Sensor Upgrade [MapMyWorld] -->
+  <joint name="camera_optical_joint" type="fixed">
+    <origin xyz="0 0 0" rpy="-1.5707 0 -1.5707"/>
+    <parent link="camera"/>
+    <child link="camera_link_optical"/>
+  </joint>
+  <link name="camera_link_optical">
+  </link>
   <!-- Lidar (hokuyo ?) -->
   <link name="hokuyo">
